File: pcb/RingOne.kicad_sch (KiCad schematic)
At the start: 0 parts

Commit message: Schema: initial placing of components
Parts:
- added C? (x2): 100nF, symbol Device:C
- added C? (x4): 100nF, Capacitor_SMD:C_0603_1608Metric, symbol Device:C
- added D?: LED_RGBA, Resistor_SMD:R_Array_Convex_2x0606, symbol Device:LED_RGBA
- added FB?: 50R@100Mhz, Inductor_SMD:L_1206_3216Metric, symbol Device:FerriteBead_Small
- added J?: USB_C_Receptacle_USB2.0, Connector_USB:USB_C_Receptacle_HRO_TYPE-C-31-M-12, symbol Connector:USB_C_Receptacle_USB2.0
- added R?: 1k, Resistor_SMD:R_0603_1608Metric, symbol Device:R
- added R? (x2): 22R, Resistor_SMD:R_0603_1608Metric, symbol Device:R
- added R?: 100k, Resistor_SMD:R_0603_1608Metric, symbol Device:R
- added SW?: RST_BTN, TCY_buttons_switches:KMT031NGJLHS, symbol Switch:SW_Push
- added TP?: VBUS, TCY_connectors:TestPoint_Pad_D0.5mm, symbol Connector:TestPoint
- added U?: LSM6DSL, Package_LGA:LGA-14_3x2.5mm_P0.5mm_LayoutBorder3x4y, symbol TCY_sensors:LSM6DSL
- added U?: STM32L452CEUx, Package_DFN_QFN:QFN-48-1EP_7x7mm_P0.5mm_EP5.6x5.6mm, symbol MCU_ST_STM32L4:STM32L452CEUx
- added U?: M24C32-FMC6TG, Package_DFN_QFN:DFN-8-1EP_3x2mm_P0.5mm_EP1.3x1.5mm, symbol Memory_EEPROM:M24C01-FDW
- added U?: KTD2026BEWE, TCY_IC:UTDFN-8-1EP_1.5x1.5mm_P0.4mm_EP0.8x1.45mm, symbol TCY_IC:KTD2026BEWE
- added U?: USBLC6-2SC6, Package_TO_SOT_SMD:SOT-23-6, symbol Power_Protection:USBLC6-2SC6
- added U?: AT25SF321B, Package_DFN_QFN:DFN-8-1EP_6x5mm_P1.27mm_EP4x4mm, symbol Memory_Flash:AT25SF081-SSHF-X
- added U?: STUSB1600AQTR, Package_DFN_QFN:QFN-24-1EP_4x4mm_P0.5mm_EP2.7x2.7mm, symbol TCY_IC:STUSB1600AQTR
- added U?: NCV8165ML330, Package_DFN_QFN:DFN-8-1EP_3x3mm_P0.65mm_EP1.55x2.4mm, symbol TCY_voltage_regulators:NCV8165ML330
Connections:
- new net: C?.1, R?.2, R?.2, SW?.1
- new net: R?.1, U?.6 (I/O1)
- new net: FB?.1, J?.S1 (SHIELD)
- new net: R?.1, U?.4 (I/O2)
- new net: D?.3 (BK), U?.2 (D3)
- new net: D?.2 (GK), U?.3 (D2)
- new net: D?.1 (RK), U?.4 (D1)
- new net: J?.A7 (D-), J?.B7 (D-), U?.1 (I/O1)
- new net: J?.A6 (D+), J?.B6 (D+), U?.3 (I/O2)
- new net +3V3: C?.1, C?.1, C?.1, C?.1, R?.1, U?.1 (VBAT), U?.1 (VO), U?.24 (VDD), U?.3 (~WP~/IO2), U?.36 (VDDUSB), U?.48 (VDD), U?.5 (VDD_IO), U?.7 (~HOLD~/IO3), U?.8 (VCC), U?.8 (VCC), U?.8 (VDD), U?.9 (VDDA)
- new net CS: U?.1 (~CS), U?.12 (MODE/CS)
- new net D+: R?.2
- new net D-: R?.2
- new net GND: C?.2, C?.2, C?.2, C?.2, C?.2, C?.2, FB?.2, J?.A1 (GND), J?.A12 (GND), J?.B1 (GND), J?.B12 (GND), SW?.2, U?.1 (E0), U?.2 (E1), U?.2 (GND), U?.2 (SDx), U?.23 (VSS), U?.3 (E2), U?.3 (SCx), U?.35 (VSS), U?.4 (GND), U?.4 (VSS), U?.47 (VSS), U?.49 (VSS), U?.6 (GND), U?.7 (GND), U?.7 (~WC), U?.8 (GND), U?.8 (VSSA), U?.9 (E_PAD)
- new net IMU_INT1: U?.4 (INT1)
- new net IMU_INT2: U?.9 (INT2)
- new net LED_PWR: C?.1, D?.4 (A), U?.5 (VIN)
- new net MISO: U?.1 (SA0/MISO), U?.2 (SO/IO1)
- new net MOSI: U?.14 (SDA/MOSI), U?.5 (SI/IO0)
- new net RESET: R?.1
- new net SCK: U?.13 (SCL/SCK), U?.6 (SCK)
- new net SCL: U?.6 (SCL), U?.6 (SCL)
- new net SDA: U?.5 (SDA), U?.7 (SDA)
- new net VBUS: J?.A4 (VBUS), J?.A9 (VBUS), J?.B4 (VBUS), J?.B9 (VBUS), TP?.1, U?.5 (VBUS)
- no-connect marks 0 -> 3
Other:
- note added: "EEPROM"
- note added: "Flash"
- note added: "LED"
- note added: "Power is managed by load switch."
- note added: "USB type-C input"
- company: (none) -> Author: Petr Malaník
- title: (none) -> RingOne
