File: pcb/BTN_Denoise.kicad_sch (KiCad schematic)
At the start: 4 parts

Commit message: Schema: finalization of schematic, break main page into hierarchical
Parts:
- removed C?: 100nF, Capacitor_SMD:C_0603_1608Metric, symbol Device:C
- removed R?: 1k, Resistor_SMD:R_0603_1608Metric, symbol Device:R
- removed TP?: TestPoint, TCY_connectors:TestPoint_Pad_D0.5mm, symbol Connector:TestPoint
- removed U?: 74LVC2G14, Package_TO_SOT_SMD:SOT-363_SC-70-6, symbol 74xGxx:74LVC2G14
Changed lines of the file:
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@@
 (kicad_sch (version 20201015) (generator eeschema)
   (paper "A4")
-  (junction (at 133.985 91.44) (diameter 1.016) (color 0 0 0 0))
-  (junction (at 153.67 91.44) (diameter 1.016) (color 0 0 0 0))
-  (wire (pts (xy 121.92 91.44) (xy 124.46 91.44))
-    (stroke (width 0) (type solid) (color 0 0 0 0))
-  )
-  (wire (pts (xy 132.08 91.44) (xy 133.985 91.44))
-    (stroke (width 0) (type solid) (color 0 0 0 0))
-  )
-  (wire (pts (xy 133.985 91.44) (xy 139.7 91.44))
-    (stroke (width 0) (type solid) (color 0 0 0 0))
-  )
-  (wire (pts (xy 158.75 91.44) (xy 153.67 91.44))
-    (stroke (width 0) (type solid) (color 0 0 0 0))
-  )
-  (hierarchical_label "IN" (shape input) (at 121.92 91.44 180)
-    (effects (font (size 1.27 1.27)) (justify right))
-  )
-  (hierarchical_label "OUT" (shape input) (at 158.75 91.44 0)
-    (effects (font (size 1.27 1.27)) (justify left))
-  )
-  (symbol (lib_id "Connector:TestPoint") (at 153.67 91.44 0)
-    (in_bom yes) (on_board yes)
-    (property "Reference" "TP?" (id 0) (at 155.575 86.995 0)
-      (effects (font (size 1.27 1.27)) (justify left))
-    )
-    (property "Value" "TestPoint" (id 1) (at 155.575 90.805 0)
-      (effects (font (size 1.27 1.27)) (justify left) hide)
-    )
-    (property "Footprint" "TCY_connectors:TestPoint_Pad_D0.5mm" (id 2) (at 158.75 91.44 0)
-      (effects (font (size 1.27 1.27)) hide)
-    )
-    (property "Datasheet" "~" (id 3) (at 158.75 91.44 0)
-      (effects (font (size 1.27 1.27)) hide)
-    )
-  )
-  (symbol (lib_id "power:VCC") (at 147.32 87.63 0)
-    (in_bom yes) (on_board yes)
-    (property "Reference" "#PWR?" (id 0) (at 147.32 91.44 0)
-      (effects (font (size 1.27 1.27)) hide)
-    )
-    (property "Value" "VCC" (id 1) (at 150.2283 85.8456 0))
-    (property "Footprint" "" (id 2) (at 147.32 87.63 0)
-      (effects (font (size 1.27 1.27)) hide)
-    )
-    (property "Datasheet" "" (id 3) (at 147.32 87.63 0)
-      (effects (font (size 1.27 1.27)) hide)
-    )
-  )
-  (symbol (lib_id "power:GND") (at 133.985 99.06 0)
-    (in_bom yes) (on_board yes)
-    (property "Reference" "#PWR?" (id 0) (at 133.985 105.41 0)
-      (effects (font (size 1.27 1.27)) hide)
-    )
-    (property "Value" "GND" (id 1) (at 133.985 102.87 0))
-    (property "Footprint" "" (id 2) (at 133.985 99.06 0)
-      (effects (font (size 1.27 1.27)) hide)
-    )
-    (property "Datasheet" "" (id 3) (at 133.985 99.06 0)
-      (effects (font (size 1.27 1.27)) hide)
-    )
-  )
-  (symbol (lib_id "power:GND") (at 147.32 95.25 0)
-    (in_bom yes) (on_board yes)
-    (property "Reference" "#PWR?" (id 0) (at 147.32 101.6 0)
-      (effects (font (size 1.27 1.27)) hide)
-    )
-    (property "Value" "GND" (id 1) (at 147.32 100.33 0))
-    (property "Footprint" "" (id 2) (at 147.32 95.25 0)
-      (effects (font (size 1.27 1.27)) hide)
-    )
-    (property "Datasheet" "" (id 3) (at 147.32 95.25 0)
-      (effects (font (size 1.27 1.27)) hide)
-    )
-  )
-  (symbol (lib_id "Device:R") (at 128.27 91.44 270)
-    (in_bom yes) (on_board yes)
-    (property "Reference" "R?" (id 0) (at 128.27 86.1822 90))
-    (property "Value" "1k" (id 1) (at 128.27 88.4936 90))
-    (property "Footprint" "Resistor_SMD:R_0603_1608Metric" (id 2) (at 128.27 89.662 90)
-      (effects (font (size 1.27 1.27)) hide)
-    )
-    (property "Datasheet" "~" (id 3) (at 128.27 91.44 0)
-      (effects (font (size 1.27 1.27)) hide)
-    )
-  )
-  (symbol (lib_id "Device:C") (at 133.985 95.25 0)
-    (in_bom yes) (on_board yes)
-    (property "Reference" "C?" (id 0) (at 136.906 94.0816 0)
-      (effects (font (size 1.27 1.27)) (justify left))
-    )
-    (property "Value" "100nF" (id 1) (at 136.906 96.393 0)
-      (effects (font (size 1.27 1.27)) (justify left))
-    )
-    (property "Footprint" "Capacitor_SMD:C_0603_1608Metric" (id 2) (at 134.9502 99.06 0)
-      (effects (font (size 1.27 1.27)) hide)
-    )
-    (property "Datasheet" "~" (id 3) (at 133.985 95.25 0)
-      (effects (font (size 1.27 1.27)) hide)
-    )
-  )
-  (symbol (lib_id "74xGxx:74LVC2G14") (at 147.32 91.44 0)
-    (in_bom yes) (on_board yes)
-    (property "Reference" "U?" (id 0) (at 151.765 93.326 0))
-    (property "Value" "74LVC2G14" (id 1) (at 154.305 95.6245 0))
-    (property "Footprint" "Package_TO_SOT_SMD:SOT-363_SC-70-6" (id 2) (at 147.32 91.44 0)
-      (effects (font (size 1.27 1.27)) hide)
-    )
-    (property "Datasheet" "https://www.ti.com/lit/ds/symlink/sn74lvc2g14.pdf" (id 3) (at 147.32 91.44 0)
-      (effects (font (size 1.27 1.27)) hide)
-    )
-  )
 )
